File: hot_plate_controller.sch (EAGLE design)
At the start: 7 parts, among them J3 B4B-PH-K-S(LF)(SN), J5 1862042, J6 1862042, J7 1862042, U1 WEMOS_LOLIN32, U2 MAX6675

Commit message: - Add MotionLab logo. - Add separated power planes on AC side. - Add high voltage symbol. - place all texts in the right side with the right rotation. - add markings for SSR, thermocouple, i2c and AC in the hot plate board. - add a second connector for AC, just in case is needed to use as bridge. - add second i2c port. - add vias to communicate power planes.
Parts:
- added J1, J2: 1862042, RE_hot_plate_controller:1862042
- J3: value B4B-PH-K-S(LF)(SN) -> 1862042; device RE_hot_plate_controller:B4B-PH-K-S(LF)(SN) -> RE_hot_plate_controller:1862042
- J5, J6: value 1862042 -> B4B-PH-K-S(LF)(SN); device RE_hot_plate_controller:1862042 -> RE_hot_plate_controller:B4B-PH-K-S(LF)(SN)
- renumbered J7 to J4
Connections:
- removed net N$1: J5.1, PS1.AC_L
- removed net N$3: J5.2, PS1.AC_N
- new net AC_L: J1.1, J2.1, PS1.AC_L
- new net AC_N: J1.2, J2.2, PS1.AC_N
- net +5V: now also J5.1, J6.1; no longer J3.1
- net GND: now also J3.2, J5.4, J6.4; no longer J3.4, J6.2
- net I2C_SCL: now also J5.3, J6.3; no longer J3.3
- net I2C_SDA: now also J5.2, J6.2; no longer J3.2
- net SSR: now also J3.1; no longer J6.1
Changed lines of the file:
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@@
 <part name="GND3" library="supply1" library_urn="urn:adsk.eagle:library:371" deviceset="GND" device=""/>
 <part name="GND4" library="supply1" library_urn="urn:adsk.eagle:library:371" deviceset="GND" device=""/>
-<part name="J3" library="RE_hot_plate_controller" deviceset="B4B-PH-K-S(LF)(SN)" device=""/>
+<part name="J5" library="RE_hot_plate_controller" deviceset="B4B-PH-K-S(LF)(SN)" device=""/>
 <part name="GND5" library="supply1" library_urn="urn:adsk.eagle:library:371" deviceset="GND" device=""/>
 <part name="P+3" library="supply1" library_urn="urn:adsk.eagle:library:371" deviceset="+5V" device=""/>
 <part name="P+4" library="supply1" library_urn="urn:adsk.eagle:library:371" deviceset="+5V" device=""/>
-<part name="J5" library="RE_hot_plate_controller" deviceset="1862042" device=""/>
-<part name="J6" library="RE_hot_plate_controller" deviceset="1862042" device=""/>
-<part name="J7" library="RE_hot_plate_controller" deviceset="1862042" device=""/>
+<part name="J1" library="RE_hot_plate_controller" deviceset="1862042" device=""/>
+<part name="J3" library="RE_hot_plate_controller" deviceset="1862042" device=""/>
+<part name="J4" library="RE_hot_plate_controller" deviceset="1862042" device=""/>
 <part name="U2" library="RE_hot_plate_controller" deviceset="MAX6675" device=""/>
 <part name="GND6" library="supply1" library_urn="urn:adsk.eagle:library:371" deviceset="GND" device=""/>
 <part name="P+5" library="supply1" library_urn="urn:adsk.eagle:library:371" deviceset="+5V" device=""/>
+<part name="J2" library="RE_hot_plate_controller" deviceset="1862042" device=""/>
+<part name="J6" library="RE_hot_plate_controller" deviceset="B4B-PH-K-S(LF)(SN)" device=""/>
+<part name="GND7" library="supply1" library_urn="urn:adsk.eagle:library:371" deviceset="GND" device=""/>
+<part name="P+6" library="supply1" library_urn="urn:adsk.eagle:library:371" deviceset="+5V" device=""/>
 </parts>
 <sheets>
@@
 <text x="223.52" y="88.9" size="1.27" layer="91">Connection for a thermocouple
 sensor</text>
+<text x="223.52" y="93.98" size="1.27" layer="91">Connection to an mlx9614
+IR temperature sensor</text>
 </plain>
 <instances>
@@
 <attribute name="VALUE" x="27.94" y="93.98" size="1.778" layer="96"/>
 </instance>
-<instance part="J3" gate="G$1" x="228.6" y="139.7" smashed="yes">
+<instance part="J5" gate="G$1" x="228.6" y="139.7" smashed="yes">
 <attribute name="NAME" x="226.05818125" y="145.800359375" size="1.77926875" layer="95"/>
 <attribute name="VALUE" x="226.05705" y="129.5282" size="1.780059375" layer="96"/>
@@
 <attribute name="VALUE" x="180.34" y="152.4" size="1.778" layer="96" rot="R90"/>
 </instance>
-<instance part="J5" gate="G$1" x="15.24" y="147.32" smashed="yes" rot="MR0">
+<instance part="J1" gate="G$1" x="15.24" y="147.32" smashed="yes" rot="MR0">
 <attribute name="NAME" x="17.78526875" y="150.501590625" size="1.27505" layer="95" rot="MR0"/>
 <attribute name="VALUE" x="17.78715" y="139.678559375" size="1.2761" layer="96" rot="MR0"/>
 </instance>
-<instance part="J6" gate="G$1" x="15.24" y="104.14" smashed="yes" rot="MR0">
+<instance part="J3" gate="G$1" x="15.24" y="104.14" smashed="yes" rot="MR0">
 <attribute name="NAME" x="17.78526875" y="107.321590625" size="1.27505" layer="95" rot="MR0"/>
 <attribute name="VALUE" x="17.78715" y="96.498559375" size="1.2761" layer="96" rot="MR0"/>
 </instance>
-<instance part="J7" gate="G$1" x="93.98" y="116.84" smashed="yes">
+<instance part="J4" gate="G$1" x="93.98" y="116.84" smashed="yes">
 <attribute name="NAME" x="91.43473125" y="120.021590625" size="1.27505" layer="95"/>
 <attribute name="VALUE" x="91.43285" y="109.198559375" size="1.2761" layer="96"/>
@@
 <instance part="P+5" gate="1" x="43.18" y="58.42" smashed="yes">
 <attribute name="VALUE" x="40.64" y="53.34" size="1.778" layer="96" rot="R90"/>
+</instance>
+<instance part="J2" gate="G$1" x="15.24" y="134.62" smashed="yes" rot="MR0">
+<attribute name="NAME" x="17.78526875" y="137.801590625" size="1.27505" layer="95" rot="MR0"/>
+<attribute name="VALUE" x="17.78715" y="126.978559375" size="1.2761" layer="96" rot="MR0"/>
+</instance>
+<instance part="J6" gate="G$1" x="228.6" y="111.76" smashed="yes">
+<attribute name="NAME" x="226.05818125" y="117.860359375" size="1.77926875" layer="95"/>
+<attribute name="VALUE" x="226.05705" y="101.5882" size="1.780059375" layer="96"/>
+</instance>
+<instance part="GND7" gate="1" x="218.44" y="101.6" smashed="yes">
+<attribute name="VALUE" x="215.9" y="99.06" size="1.778" layer="96"/>
+</instance>
+<instance part="P+6" gate="1" x="218.44" y="119.38" smashed="yes">
+<attribute name="VALUE" x="215.9" y="114.3" size="1.778" layer="96" rot="R90"/>
 </instance>
 </instances>
@@
 </busses>
 <nets>
-<net name="N$1" class="0">
+<net name="AC_L" class="0">
 <segment>
 <pinref part="PS1" gate="G$1" pin="AC_L"/>
-<wire x1="22.86" y1="147.32" x2="27.94" y2="147.32" width="0.1524" layer="91"/>
+<wire x1="22.86" y1="147.32" x2="25.4" y2="147.32" width="0.1524" layer="91"/>
+<wire x1="25.4" y1="147.32" x2="27.94" y2="147.32" width="0.1524" layer="91"/>
 <wire x1="27.94" y1="147.32" x2="27.94" y2="149.86" width="0.1524" layer="91"/>
 <wire x1="27.94" y1="149.86" x2="33.02" y2="149.86" width="0.1524" layer="91"/>
-<pinref part="J5" gate="G$1" pin="1"/>
-</segment>
-</net>
-<net name="N$3" class="0">
+<pinref part="J1" gate="G$1" pin="1"/>
+<pinref part="J2" gate="G$1" pin="1"/>
+<wire x1="22.86" y1="134.62" x2="25.4" y2="134.62" width="0.1524" layer="91"/>
+<wire x1="25.4" y1="134.62" x2="25.4" y2="147.32" width="0.1524" layer="91"/>
+<junction x="25.4" y="147.32"/>
+</segment>
+</net>
+<net name="AC_N" class="0">
 <segment>
 <pinref part="PS1" gate="G$1" pin="AC_N"/>
@@
 <wire x1="27.94" y1="144.78" x2="27.94" y2="139.7" width="0.1524" layer="91"/>
 <wire x1="27.94" y1="139.7" x2="33.02" y2="139.7" width="0.1524" layer="91"/>
-<pinref part="J5" gate="G$1" pin="2"/>
+<pinref part="J1" gate="G$1" pin="2"/>
+<pinref part="J2" gate="G$1" pin="2"/>
+<wire x1="22.86" y1="132.08" x2="27.94" y2="132.08" width="0.1524" layer="91"/>
+<wire x1="27.94" y1="132.08" x2="27.94" y2="139.7" width="0.1524" layer="91"/>
+<junction x="27.94" y="139.7"/>
 </segment>
 </net>
@@
 <wire x1="30.48" y1="101.6" x2="30.48" y2="99.06" width="0.1524" layer="91"/>
 <pinref part="GND4" gate="1" pin="GND"/>
-<pinref part="J6" gate="G$1" pin="2"/>
-</segment>
-<segment>
-<pinref part="J3" gate="G$1" pin="4"/>
+<pinref part="J3" gate="G$1" pin="2"/>
+</segment>
+<segment>
+<pinref part="J5" gate="G$1" pin="4"/>
 <wire x1="220.98" y1="134.62" x2="218.44" y2="134.62" width="0.1524" layer="91"/>
 <wire x1="218.44" y1="134.62" x2="218.44" y2="132.08" width="0.1524" layer="91"/>
@@
 <pinref part="GND6" gate="1" pin="GND"/>
 </segment>
+<segment>
+<pinref part="J6" gate="G$1" pin="4"/>
+<wire x1="220.98" y1="106.68" x2="218.44" y2="106.68" width="0.1524" layer="91"/>
+<wire x1="218.44" y1="106.68" x2="218.44" y2="104.14" width="0.1524" layer="91"/>
+<pinref part="GND7" gate="1" pin="GND"/>
+</segment>
 </net>
 <net name="+5V" class="0">
@@
 </segment>
 <segment>
-<pinref part="J3" gate="G$1" pin="1"/>
+<pinref part="J5" gate="G$1" pin="1"/>
 <wire x1="220.98" y1="142.24" x2="218.44" y2="142.24" width="0.1524" layer="91"/>
 <wire x1="218.44" y1="142.24" x2="218.44" y2="144.78" width="0.1524" layer="91"/>
@@
 <pinref part="P+5" gate="1" pin="+5V"/>
 </segment>
+<segment>
+<pinref part="J6" gate="G$1" pin="1"/>
+<wire x1="220.98" y1="114.3" x2="218.44" y2="114.3" width="0.1524" layer="91"/>
+<wire x1="218.44" y1="114.3" x2="218.44" y2="116.84" width="0.1524" layer="91"/>
+<pinref part="P+6" gate="1" pin="+5V"/>
+</segment>
 </net>
 <net name="I2C_SCL" class="0">
@@
 </segment>
 <segment>
-<pinref part="J3" gate="G$1" pin="3"/>
+<pinref part="J5" gate="G$1" pin="3"/>
 <wire x1="220.98" y1="137.16" x2="218.44" y2="137.16" width="0.1524" layer="91"/>
 <label x="218.44" y="137.16" size="1.27" layer="95" rot="R180" xref="yes"/>
+</segment>
+<segment>
+<pinref part="J6" gate="G$1" pin="3"/>
+<wire x1="220.98" y1="109.22" x2="218.44" y2="109.22" width="0.1524" layer="91"/>
+<label x="218.44" y="109.22" size="1.27" layer="95" rot="R180" xref="yes"/>
 </segment>
 </net>
@@
 </segment>
 <segment>
-<pinref part="J3" gate="G$1" pin="2"/>
+<pinref part="J5" gate="G$1" pin="2"/>
 <wire x1="220.98" y1="139.7" x2="218.44" y2="139.7" width="0.1524" layer="91"/>
 <label x="218.44" y="139.7" size="1.27" layer="95" rot="R180" xref="yes"/>
+</segment>
+<segment>
+<pinref part="J6" gate="G$1" pin="2"/>
+<wire x1="220.98" y1="111.76" x2="218.44" y2="111.76" width="0.1524" layer="91"/>
+<label x="218.44" y="111.76" size="1.27" layer="95" rot="R180" xref="yes"/>
 </segment>
 </net>
@@
 <wire x1="22.86" y1="104.14" x2="30.48" y2="104.14" width="0.1524" layer="91"/>
 <label x="30.48" y="104.14" size="1.27" layer="95" xref="yes"/>
-<pinref part="J6" gate="G$1" pin="1"/>
+<pinref part="J3" gate="G$1" pin="1"/>
 </segment>
 </net>
@@
 </segment>
 <segment>
-<pinref part="J7" gate="G$1" pin="2"/>
+<pinref part="J4" gate="G$1" pin="2"/>
 <wire x1="86.36" y1="114.3" x2="83.82" y2="114.3" width="0.1524" layer="91"/>
 <label x="83.82" y="114.3" size="1.27" layer="95" rot="R180" xref="yes"/>
@@
 </segment>
 <segment>
-<pinref part="J7" gate="G$1" pin="1"/>
+<pinref part="J4" gate="G$1" pin="1"/>
 <wire x1="86.36" y1="116.84" x2="83.82" y2="116.84" width="0.1524" layer="91"/>
 <label x="83.82" y="116.84" size="1.27" layer="95" rot="R180" xref="yes"/>
